Commit message: feat(ik): complete Phase 5 analytical inverse kinematics and vision reaching pipeline
- Implement closed-form analytical 5-DOF IK solver in nova_ik.hpp with top-down and horizontal reach support
- Fix static camera TF orientation in sim_and_rviz.launch.py to align optical frame with table workspace
- Align arm base orientation in URDF and scene.xml
- Update object_detector_node with dual-range HSV red cube detection and 3D back-projection
- Integrate ik_solver_node with live perception and joint controller
- Add standalone IK verification tools

File: src/nova_description/urdf/diy_6dof_arm.urdf (robot description, URDF)
Before this commit: robot diy_6dof_arm, 10 links, 9 joints
Joints:
- joint joint1: origin xyz=0 0 0.02 rpy=0 0 0 -> xyz=0 0 0.02 rpy=0 0 1.5708
